Commit message: Added pose task.

File: models/dofarm/dofarm.urdf (robot description, URDF)
Before this commit: robot dofarm_description, 7 links, 6 joints
Links:
- added link ee, mass 0.11; collision mesh filename=package://dofarm/ee.stl scale=0.001 0.001 0.001; visual mesh filename=package://dofarm/ee.stl scale=0.001 0.001 0.001
- added link wrist3, mass 0.11; collision mesh filename=package://dofarm/ee_wrist.stl scale=0.001 0.001 0.001; visual mesh filename=package://dofarm/ee_wrist.stl scale=0.001 0.001 0.001
Joints:
- added joint wrist2_wrist3: type revolute, parent wrist2, child wrist3, origin xyz=0 0 0.12 rpy=0 0 0, axis 0 0 1, limit lower=-3.14 upper=3.14 effort=100 velocity=20
- added joint wrist3_ee: type fixed, parent wrist3, child ee, origin xyz=0 0 0.047 rpy=0 0 0
- joint arm_forearm: limit lower=-3.14 upper=3.14 effort=100 velocity=20 -> lower=-1.57 upper=1.57 effort=100 velocity=20
- joint waist_shoulder: limit lower=-3.14 upper=3.14 effort=100 velocity=20 -> lower=-1.57 upper=1.57 effort=100 velocity=20
- joint wrist_wrist2: limit lower=-3.14 upper=3.14 effort=100 velocity=20 -> lower=-1.57 upper=1.57 effort=100 velocity=20

Commit message: Added kinova arm and fixed joint tasks

File: models/dofarm/dofarm.urdf (robot description, URDF)
Before this commit: robot dofarm_description, 9 links, 8 joints
Links:
- removed link ee
- added link vx300s/ee_arm_link, mass 0.001
- added link vx300s/ee_gripper_link, mass 0.001
- added link vx300s/fingers_link, mass 0.001
- added link vx300s/gripper_bar_link, mass 0.150986; collision mesh filename=package://dofarm/vx300s_9_gripper_bar.stl scale=0.001 0.001 0.001; visual mesh filename=package://dofarm/vx300s_9_gripper_bar.stl scale=0.001 0.001 0.001
- added link vx300s/gripper_link, mass 0.097666; collision mesh filename=package://dofarm/vx300s_7_gripper.stl scale=0.001 0.001 0.001; visual mesh filename=package://dofarm/vx300s_7_gripper.stl scale=0.001 0.001 0.001
- added link vx300s/gripper_prop_link, mass 0.008009; collision mesh filename=package://dofarm/vx300s_8_gripper_prop.stl scale=0.001 0.001 0.001; visual mesh filename=package://dofarm/vx300s_8_gripper_prop.stl scale=0.001 0.001 0.001
- added link vx300s/left_finger_link, mass 0.034796; collision mesh filename=package://dofarm/vx300s_10_gripper_finger.stl scale=0.001 0.001 0.001; visual mesh filename=package://dofarm/vx300s_10_gripper_finger.stl scale=0.001 0.001 0.001
- added link vx300s/right_finger_link, mass 0.034796; collision mesh filename=package://dofarm/vx300s_10_gripper_finger.stl scale=0.001 0.001 0.001; visual mesh filename=package://dofarm/vx300s_10_gripper_finger.stl scale=0.001 0.001 0.001
Joints:
- added joint ee_arm: type fixed, parent vx300s/gripper_link, child vx300s/ee_arm_link, origin xyz=0.042825 0 0 rpy=0 0 0, axis 1 0 0
- added joint ee_bar: type fixed, parent vx300s/gripper_bar_link, child vx300s/fingers_link, origin xyz=0.025875 0 0 rpy=0 0 0, axis 1 0 0
- added joint ee_gripper: type fixed, parent vx300s/fingers_link, child vx300s/ee_gripper_link, origin xyz=0.0385 0 0 rpy=0 0 0, axis 1 0 0
- added joint gripper: type fixed, parent vx300s/ee_arm_link, child vx300s/gripper_prop_link, origin xyz=0.005675 0 0 rpy=0 0 0, axis 1 0 0, limit effort=1 velocity=3.141592653589793
- added joint gripper_bar: type fixed, parent vx300s/ee_arm_link, child vx300s/gripper_bar_link, origin xyz=0 0 0 rpy=0 0 0, axis 1 0 0
- added joint left_finger: type prismatic, parent vx300s/fingers_link, child vx300s/left_finger_link, origin xyz=0 0 0 rpy=0 0 0, axis 0 1 0, limit lower=0.021 upper=0.057 effort=5 velocity=1
- added joint right_finger: type prismatic, parent vx300s/fingers_link, child vx300s/right_finger_link, origin xyz=0 0 0 rpy=0 0 0, axis 0 1 0, limit lower=-0.057 upper=-0.021 effort=5 velocity=1, mimic joint=left_finger multiplier=-1 offset=0
- joint arm_forearm: limit lower=-1.57 upper=1.57 effort=100 velocity=20 -> lower=-1.57 upper=1.57 effort=100 velocity=3.14
- joint base_waist: limit lower=-3.14 upper=3.14 effort=100 velocity=20 -> lower=-3.14 upper=3.14 effort=100 velocity=3.14
- joint forearm_wrist: limit lower=-3.14 upper=3.14 effort=100 velocity=20 -> lower=-3.14 upper=3.14 effort=100 velocity=3.14
- joint shoulder_arm: limit lower=-3.14 upper=3.14 effort=100 velocity=20 -> lower=-3.14 upper=3.14 effort=100 velocity=3.14
- joint waist_shoulder: limit lower=-1.57 upper=1.57 effort=100 velocity=20 -> lower=-1.57 upper=1.57 effort=100 velocity=3.14
- joint wrist2_wrist3: limit lower=-3.14 upper=3.14 effort=100 velocity=20 -> lower=-3.14 upper=3.14 effort=100 velocity=3.14
- joint wrist3_ee: child ee -> vx300s/gripper_link; origin xyz=0 0 0.047 rpy=0 0 0 -> xyz=0 0 0.047 rpy=0 -1.57 0
- joint wrist_wrist2: limit lower=-1.57 upper=1.57 effort=100 velocity=20 -> lower=-1.57 upper=1.57 effort=100 velocity=3.14

Commit message: using quaternions for Cartesian task and fixed gain error.

File: models/dofarm/dofarm.urdf (robot description, URDF)
Before this commit: robot dofarm_description, 16 links, 15 joints
Joints:
- joint arm_forearm: limit lower=-1.57 upper=1.57 effort=100 velocity=3.14 -> lower=-2.23 upper=2.23 effort=9 velocity=0.8727
- joint base_waist: limit lower=-3.14 upper=3.14 effort=100 velocity=3.14 -> lower=-3.14 upper=3.14 effort=100 velocity=0.8727
- joint forearm_wrist: limit lower=-3.14 upper=3.14 effort=100 velocity=3.14 -> lower=-3.14 upper=3.14 effort=100 velocity=0.8727
- joint shoulder_arm: limit lower=-3.14 upper=3.14 effort=100 velocity=3.14 -> lower=-3.14 upper=3.14 effort=100 velocity=0.8727
- joint waist_shoulder: limit lower=-1.57 upper=1.57 effort=100 velocity=3.14 -> lower=-2.23 upper=2.23 effort=9 velocity=0.8727
- joint wrist2_wrist3: limit lower=-3.14 upper=3.14 effort=100 velocity=3.14 -> lower=-3.14 upper=3.14 effort=100 velocity=0.8727
- joint wrist_wrist2: limit lower=-1.57 upper=1.57 effort=100 velocity=3.14 -> lower=-2.23 upper=2.23 effort=9 velocity=0.8727
